File: Clock/Clock.kicad_pcb (KiCad board)
At the start: 2 copper layers, 99.6 x 59.9 mm, 37 parts, among them J1 Conn_01x16, J2 Conn_01x16, SW1 SW_Push, SW2 SW_Push, SW3 SW_Push, SW4 SW_Push, U1 74LS02, U2 74LS32, U4 74LS08, U5 LM555xN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

Commit message: Update all boards to r3, and update revision log and gitignore
Parts:
- added HOLE1: MountingHole_2.2mm_M2_DIN965_Pad, MountingHole:MountingHole_2.2mm_M2_DIN965_Pad, F.Cu at (35.6, 38.1)
- added HOLE2: MountingHole_2.2mm_M2_DIN965_Pad, MountingHole:MountingHole_2.2mm_M2_DIN965_Pad, F.Cu at (127.0, 38.1)
- added HOLE3: MountingHole_2.2mm_M2_DIN965_Pad, MountingHole:MountingHole_2.2mm_M2_DIN965_Pad, F.Cu at (35.6, 89.9)
- added HOLE4: MountingHole_2.2mm_M2_DIN965_Pad, MountingHole:MountingHole_2.2mm_M2_DIN965_Pad, F.Cu at (127.0, 89.9)
- RV1: value 100k -> 1M; footprint Potentiometer_THT:Potentiometer_Alps_RK09Y11_Single_Horizontal -> Potentiometer_THT:Potentiometer_Bourns_PTV09A-1_Single_Vertical
- U1: value 74LS02 -> 74HC02
- U2, U6: value 74LS32 -> 74HC32
- U4: value 74LS08 -> 74HC08
- moved C8 74.5 mm to (46.2, 44.5), turned to -90 degrees
- moved U2 64.2 mm to (49.3, 51.1), turned to 90 degrees
- moved C7 59.7 mm to (46.2, 55.4), turned to -90 degrees
- moved RV1 54.5 mm to (105.3, 83.7)
- moved C1 53.1 mm to (110.0, 71.4)
- moved C2 53.1 mm to (110.0, 68.3)
- moved D4 53.1 mm to (98.3, 88.6)
- moved R5 53.1 mm to (98.8, 84.1)
- moved U5 53.1 mm to (98.3, 63.2)
- moved R4 53.1 mm to (109.0, 64.8)
- moved U1 49.7 mm to (49.3, 62.0), turned to 90 degrees
- moved C3 32.8 mm to (50.0, 83.6)
- moved R6 32.8 mm to (45.5, 70.4)
- moved R7 32.8 mm to (58.7, 70.4)
- moved SW4 32.8 mm to (59.2, 74.9)
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Connections:
- J1 pad 10: Net-(J1-Pad10) -> unconnected-(J1-Pin_10-Pad10)
- J1 pad 11: Net-(J1-Pad11) -> unconnected-(J1-Pin_11-Pad11)
- J1 pad 12: Net-(J1-Pad12) -> unconnected-(J1-Pin_12-Pad12)
- J1 pad 13: Net-(J1-Pad13) -> unconnected-(J1-Pin_13-Pad13)
- J1 pad 14: Net-(J1-Pad14) -> unconnected-(J1-Pin_14-Pad14)
- J1 pad 15: Net-(J1-Pad15) -> unconnected-(J1-Pin_15-Pad15)
- J1 pad 16: Net-(J1-Pad16) -> unconnected-(J1-Pin_16-Pad16)
- J1 pad 5: Net-(J1-Pad5) -> unconnected-(J1-Pin_5-Pad5)
- J1 pad 6: Net-(J1-Pad6) -> unconnected-(J1-Pin_6-Pad6)
- J1 pad 7: Net-(J1-Pad7) -> unconnected-(J1-Pin_7-Pad7)
- J1 pad 8: Net-(J1-Pad8) -> unconnected-(J1-Pin_8-Pad8)
- J1 pad 9: Net-(J1-Pad9) -> unconnected-(J1-Pin_9-Pad9)
- J2 pad 1: Net-(J2-Pad1) -> unconnected-(J2-Pin_1-Pad1)
- J2 pad 10: Net-(J2-Pad10) -> unconnected-(J2-Pin_10-Pad10)
- J2 pad 11: Net-(J2-Pad11) -> unconnected-(J2-Pin_11-Pad11)
- J2 pad 12: Net-(J2-Pad12) -> unconnected-(J2-Pin_12-Pad12)
- J2 pad 2: Net-(J2-Pad2) -> unconnected-(J2-Pin_2-Pad2)
- J2 pad 3: Net-(J2-Pad3) -> unconnected-(J2-Pin_3-Pad3)
- J2 pad 4: Net-(J2-Pad4) -> unconnected-(J2-Pin_4-Pad4)
- J2 pad 5: Net-(J2-Pad5) -> unconnected-(J2-Pin_5-Pad5)
- J2 pad 6: Net-(J2-Pad6) -> unconnected-(J2-Pin_6-Pad6)
- J2 pad 7: Net-(J2-Pad7) -> unconnected-(J2-Pin_7-Pad7)
- J2 pad 8: Net-(J2-Pad8) -> unconnected-(J2-Pin_8-Pad8)
- J2 pad 9: Net-(J2-Pad9) -> unconnected-(J2-Pin_9-Pad9)
- RV1 pad 3: Net-(RV1-Pad3) -> unconnected-(RV1-Pad3)
- U1 pad 13: Net-(U1-Pad13) -> unconnected-(U1-Pad13)
- U4 pad 11: Net-(U4-Pad11) -> unconnected-(U4-Pad11)
- U6 pad 11: Net-(U6-Pad11) -> unconnected-(U6-Pad11)
- U6 pad 8: Net-(U6-Pad8) -> unconnected-(U6-Pad8)
- X1 pad 1: Net-(X1-Pad1) -> unconnected-(X1-NC-Pad1)
Routing:
- net Net-(R3-Pad2): track 26.3 -> 80.6 mm
- net Net-(D4-K): track 11.9 -> 56.6 mm
- net GND: track 256.9 -> 220.7 mm
- net Net-(D4-A): track 72.9 -> 37.1 mm
- net GND_1k: track 98.9 -> 64.0 mm
- net Net-(R2-Pad2): track 31.0 -> 62.3 mm
- net Net-(R1-Pad2): track 28.6 -> 59.8 mm
- net Net-(D5-K): track 98.3 -> 73.1 mm, vias 0 -> 1
- net Net-(D2-K): track 51.1 -> 30.5 mm, vias 0 -> 1
- net RESET: track 119.9 -> 103.5 mm
- net Net-(D6-K): track 19.5 -> 35.7 mm
- net Net-(D3-A): track 100.6 -> 85.1 mm, vias 0 -> 1
- net Net-(D1-A): track 101.9 -> 90.9 mm
- net Net-(D5-A): track 96.7 -> 105.9 mm
- net Net-(D7-K): track 38.7 -> 29.6 mm
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Other:
- net class Default removed
