File: Input/Input.kicad_pcb (KiCad board)
At the start: 2 copper layers, 99.6 x 59.9 mm, 19 parts, among them J1 Conn_01x16, J2 Conn_01x16, J3 Conn_01x14, U1 74LS00, U2 74LS273, U3 74LS245

Commit message: Update all boards to r3, and update revision log and gitignore
Parts:
- added C4: 100nF, Capacitor_THT:C_Disc_D4.3mm_W1.9mm_P5.00mm, F.Cu at (113.2, 50.3)
- added HOLE1: MountingHole_2.2mm_M2_DIN965_Pad, MountingHole:MountingHole_2.2mm_M2_DIN965_Pad, F.Cu at (35.6, 38.1)
- added HOLE2: MountingHole_2.2mm_M2_DIN965_Pad, MountingHole:MountingHole_2.2mm_M2_DIN965_Pad, F.Cu at (127.0, 38.1)
- added HOLE3: MountingHole_2.2mm_M2_DIN965_Pad, MountingHole:MountingHole_2.2mm_M2_DIN965_Pad, F.Cu at (35.6, 89.9)
- added HOLE4: MountingHole_2.2mm_M2_DIN965_Pad, MountingHole:MountingHole_2.2mm_M2_DIN965_Pad, F.Cu at (127.0, 89.9)
- added U4: 74HC173, Package_DIP:DIP-16_W7.62mm, F.Cu at (106.7, 53.3)
- U1: value 74LS00 -> 74HC04
- U2: value 74LS273 -> 74HC173; footprint Package_DIP:DIP-20_W7.62mm -> Package_DIP:DIP-16_W7.62mm
- U3: value 74LS245 -> 74HC245
- moved U2 0.24 mm to (79.2, 53.3)
- moved U3 0.24 mm to (93.0, 53.3)
Connections:
- D1 pad 2: Net-(D1-Pad2) -> Net-(D1-A)
- D2 pad 2: Net-(D2-Pad2) -> Net-(D2-A)
- D3 pad 2: Net-(D3-Pad2) -> Net-(D3-A)
- D4 pad 2: Net-(D4-Pad2) -> Net-(D4-A)
- D5 pad 2: Net-(D5-Pad2) -> Net-(D5-A)
- D6 pad 2: Net-(D6-Pad2) -> Net-(D6-A)
- D7 pad 2: Net-(D7-Pad2) -> Net-(D7-A)
- D8 pad 2: Net-(D8-Pad2) -> Net-(D8-A)
- J3 pad 10: Net-(J3-Pad10) -> Net-(J3-Pin_10)
- J3 pad 11: Net-(J3-Pad11) -> Net-(J3-Pin_11)
- J3 pad 12: Net-(J3-Pad12) -> Net-(J3-Pin_12)
- J3 pad 5: Net-(J3-Pad5) -> Net-(J3-Pin_5)
- J3 pad 6: Net-(J3-Pad6) -> Net-(J3-Pin_6)
- J3 pad 7: Net-(J3-Pad7) -> Net-(J3-Pin_7)
- J3 pad 8: Net-(J3-Pad8) -> Net-(J3-Pin_8)
- J3 pad 9: Net-(J3-Pad9) -> Net-(J3-Pin_9)
- RN2 pad 2: Net-(J3-Pad12) -> Net-(J3-Pin_12)
- RN2 pad 3: Net-(J3-Pad11) -> Net-(J3-Pin_11)
- RN2 pad 4: Net-(J3-Pad10) -> Net-(J3-Pin_10)
- RN2 pad 5: Net-(J3-Pad9) -> Net-(J3-Pin_9)
- RN2 pad 6: Net-(J3-Pad8) -> Net-(J3-Pin_8)
- RN2 pad 7: Net-(J3-Pad7) -> Net-(J3-Pin_7)
- RN2 pad 8: Net-(J3-Pad6) -> Net-(J3-Pin_6)
- RN2 pad 9: Net-(J3-Pad5) -> Net-(J3-Pin_5)
- U1 pad 1: CLOCK -> SIG_OUT
- U1 pad 10: RESET -> unconnected-(U1-Pad10)
- U1 pad 11: ~SIG_OUT -> GND
- U1 pad 12: SIG_OUT -> unconnected-(U1-Pad12)
- U1 pad 13: SIG_OUT -> GND
- U1 pad 2: SIG_IN -> ~{SIG_OUT}
- U1 pad 3: Net-(U1-Pad3) -> SIG_IN
- U1 pad 4: Net-(U1-Pad3) -> ~{SIG_IN}
- U1 pad 5: Net-(U1-Pad3) -> GND
- U1 pad 6: Net-(U1-Pad6) -> unconnected-(U1-Pad6)
- U1 pad 8: Net-(U1-Pad8) -> unconnected-(U1-Pad8)
- U1 pad 9: RESET -> GND
- U2 pad 1: Net-(U1-Pad8) -> GND
- U2 pad 10: GND -> ~{SIG_IN}
- U2 pad 11: Net-(U1-Pad6) -> Net-(J3-Pin_8)
- U2 pad 12: Net-(D5-Pad2) -> Net-(J3-Pin_7)
- U2 pad 13: Net-(J3-Pad9) -> Net-(J3-Pin_6)
- U2 pad 14: Net-(J3-Pad10) -> Net-(J3-Pin_5)
- U2 pad 15: Net-(D6-Pad2) -> RESET
- U2 pad 16: Net-(D7-Pad2) -> VCC
- U2 pad 2: Net-(D1-Pad2) -> GND
- U2 pad 3: Net-(J3-Pad5) -> Net-(D8-A)
- U2 pad 4: Net-(J3-Pad6) -> Net-(D7-A)
- U2 pad 5: Net-(D2-Pad2) -> Net-(D6-A)
- U2 pad 6: Net-(D3-Pad2) -> Net-(D5-A)
- U2 pad 7: Net-(J3-Pad7) -> CLOCK
- U2 pad 8: Net-(J3-Pad8) -> GND
- U2 pad 9: Net-(D4-Pad2) -> ~{SIG_IN}
- U3 pad 19: ~SIG_OUT -> ~{SIG_OUT}
- U3 pad 2: Net-(D1-Pad2) -> Net-(D8-A)
- U3 pad 3: Net-(D2-Pad2) -> Net-(D7-A)
- U3 pad 4: Net-(D3-Pad2) -> Net-(D6-A)
- U3 pad 5: Net-(D4-Pad2) -> Net-(D5-A)
- U3 pad 6: Net-(D5-Pad2) -> Net-(D4-A)
- U3 pad 7: Net-(D6-Pad2) -> Net-(D3-A)
- U3 pad 8: Net-(D7-Pad2) -> Net-(D2-A)
- U3 pad 9: Net-(D8-Pad2) -> Net-(D1-A)
Routing:
- net Net-(J3-Pad12): track 110.9 -> 0.00 mm
- net Net-(J3-Pin_11): track 0.00 -> 109.4 mm, vias 0 -> 1
- net Net-(J3-Pin_12): track 0.00 -> 103.2 mm, vias 0 -> 1
- net Net-(J3-Pin_10): track 0.00 -> 95.0 mm, vias 0 -> 1
- net Net-(J3-Pin_9): track 0.00 -> 84.1 mm
- net ~{SIG_IN}: track 0.00 -> 84.1 mm, vias 0 -> 2
- net Net-(J3-Pad9): track 70.2 -> 0.00 mm
- net Net-(J3-Pad7): track 70.1 -> 0.00 mm
- net Net-(J3-Pad11): track 67.3 -> 0.00 mm
- net Net-(J3-Pad10): track 64.8 -> 0.00 mm
- net Net-(J3-Pad8): track 58.9 -> 0.00 mm, vias 1 -> 0
- net Net-(J3-Pin_8): track 0.00 -> 57.8 mm
- net Net-(J3-Pin_7): track 0.00 -> 55.9 mm
- net Net-(J3-Pin_6): track 0.00 -> 54.2 mm, vias 0 -> 1
- net Net-(J3-Pad6): track 52.3 -> 0.00 mm, vias 1 -> 0
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Other:
- net class Default removed
