File: RAM/RAM.kicad_pcb (KiCad board)
At the start: 2 copper layers, 99.6 x 59.9 mm, 19 parts, among them J1 Conn_01x16, J2 Conn_01x16, J3 Conn_01x16, J4 Conn_01x16, U1 HM62256BLP, U2 74LS02, U3 74LS245

Commit message: Fixed floating inputs; improved power; added parts list; replaced JK latches
Parts:
- added R1: 10k, Resistor_THT:R_Axial_DIN0207_L6.3mm_D2.5mm_P7.62mm_Horizontal, F.Cu at (125.7, 39.4)
- added RN2: 10k, Resistor_THT:R_Array_SIP9, F.Cu at (93.6, 69.2)
- RN1: value R_Network08_US -> 1k
Connections:
- U2 pad 10: (no net) -> Net-(U2-Pad10)
- U2 pad 11: (no net) -> Net-(R1-Pad2)
- U2 pad 12: (no net) -> Net-(R1-Pad2)
- U2 pad 13: (no net) -> Net-(U2-Pad13)
- U2 pad 8: (no net) -> Net-(R1-Pad2)
- U2 pad 9: (no net) -> Net-(R1-Pad2)
Routing:
- net A11: track 83.7 -> 151.1 mm, vias 2 -> 0
- net A4: track 53.3 -> 118.1 mm
- net A3: track 54.9 -> 116.4 mm
- net A1: track 53.6 -> 114.8 mm
- net Net-(R1-Pad2): track 0.00 -> 47.7 mm, vias 0 -> 1
- net A2: track 80.3 -> 114.7 mm
- net A7: track 85.6 -> 55.9 mm
- net A5: track 94.4 -> 119.8 mm, vias 1 -> 0
- net Net-(D2-Pad2): track 69.9 -> 92.7 mm, vias 1 -> 0
- net VCC: track 113.7 -> 134.7 mm, vias 0 -> 1
- net Net-(D4-Pad2): track 81.6 -> 64.1 mm, vias 0 -> 2
- net SIG_OUT: track 111.0 -> 97.1 mm
- net CLOCK: track 105.5 -> 92.0 mm
- net RESET: track 103.4 -> 114.2 mm
- net Net-(D3-Pad2): track 84.9 -> 76.5 mm, vias 0 -> 2
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
Commit message: Revise control and RAM modules
- Change control signals on low going clock
- Pull down control signals with 1k resistors
- AND the write signal with clock on RAM / ROM module
Parts:
- added C4: 100nF, Capacitor_THT:C_Disc_D4.3mm_W1.9mm_P5.00mm, F.Cu at (115.8, 68.1)
- added U4: 74LS00, Package_DIP:DIP-14_W7.62mm, F.Cu at (109.2, 71.1)
- R1: value 10k -> 1k
- moved R1 6.97 mm to (118.9, 38.1), turned to 0 degrees
Connections:
- R1 pad 1: VCC -> Net-(R1-Pad1)
- R1 pad 2: Net-(R1-Pad2) -> GND
- U1 pad 27: ~SIG_IN -> ~WE_CLOCK
- U2 pad 11: Net-(R1-Pad2) -> Net-(R1-Pad1)
- U2 pad 12: Net-(R1-Pad2) -> Net-(R1-Pad1)
- U2 pad 8: Net-(R1-Pad2) -> Net-(R1-Pad1)
- U2 pad 9: Net-(R1-Pad2) -> Net-(R1-Pad1)
Routing:
- net Net-(R1-Pad1): track 0.00 -> 77.0 mm
- net A11: track 151.1 -> 86.1 mm
- net A5: track 119.8 -> 55.4 mm
- net A4: track 118.1 -> 57.0 mm
- net A2: track 114.7 -> 54.9 mm
- net Net-(R1-Pad2): track 47.7 -> 0.00 mm, vias 1 -> 0
- net VCC: track 134.7 -> 180.0 mm, vias 1 -> 0
- net A6: track 98.1 -> 54.9 mm
- net A1: track 114.8 -> 76.8 mm
- net GND: track 184.3 -> 221.5 mm
- net ~WE_CLOCK: track 0.00 -> 34.3 mm, vias 0 -> 1
- net SIG1: track 98.1 -> 126.2 mm
- net A3: track 116.4 -> 89.1 mm
- net ~SIG_IN: track 37.8 -> 11.6 mm
- net CLOCK: track 92.0 -> 118.1 mm, vias 0 -> 1
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
Commit message: Update all boards to r3, and update revision log and gitignore
Parts:
- removed R1: 1k, Resistor_THT:R_Axial_DIN0207_L6.3mm_D2.5mm_P7.62mm_Horizontal
- added HOLE1: MountingHole_2.2mm_M2_DIN965_Pad, MountingHole:MountingHole_2.2mm_M2_DIN965_Pad, F.Cu at (35.6, 38.1)
- added HOLE2: MountingHole_2.2mm_M2_DIN965_Pad, MountingHole:MountingHole_2.2mm_M2_DIN965_Pad, F.Cu at (127.0, 38.1)
- added HOLE3: MountingHole_2.2mm_M2_DIN965_Pad, MountingHole:MountingHole_2.2mm_M2_DIN965_Pad, F.Cu at (35.6, 89.9)
- added HOLE4: MountingHole_2.2mm_M2_DIN965_Pad, MountingHole:MountingHole_2.2mm_M2_DIN965_Pad, F.Cu at (127.0, 89.9)
- added J5: 3183-10200P1T, updated_libs:318310200P1T, F.Cu at (43.5, 74.6)
- U2: value 74LS02 -> 74HC02
- U3: value 74LS245 -> 74HC245
- U4: value 74LS00 -> 74HC00
- moved U2 24.4 mm to (110.2, 71.1)
- moved U4 24.4 mm to (109.7, 46.7)
- moved D1 6.78 mm to (68.6, 79.8)
- moved D2 6.78 mm to (73.7, 79.8)
- moved D3 6.78 mm to (78.7, 79.8)
- moved D4 6.78 mm to (83.8, 79.8)
- moved D5 6.78 mm to (88.9, 79.8)
- moved D6 6.78 mm to (94.0, 79.8)
- moved D7 6.78 mm to (99.1, 79.8)
- moved D8 6.78 mm to (104.1, 79.8)
- moved RN1 6.78 mm to (97.5, 83.8)
- moved U1 2.03 mm to (83.3, 46.7)
- moved C2 0.51 mm to (116.3, 43.7)
- moved C4 0.51 mm to (116.3, 68.1)
Connections:
- net ~ENABLE renamed ~{ENABLE}
- net ~SIG_IN renamed ~{SIG_IN}
- net ~WE_CLOCK renamed ~{WE_CLOCK}
- D1 pad 2: Net-(D1-Pad2) -> Net-(D1-A)
- D2 pad 2: Net-(D2-Pad2) -> Net-(D2-A)
- D3 pad 2: Net-(D3-Pad2) -> Net-(D3-A)
- D4 pad 2: Net-(D4-Pad2) -> Net-(D4-A)
- D5 pad 2: Net-(D5-Pad2) -> Net-(D5-A)
- D6 pad 2: Net-(D6-Pad2) -> Net-(D6-A)
- D7 pad 2: Net-(D7-Pad2) -> Net-(D7-A)
- D8 pad 2: Net-(D8-Pad2) -> Net-(D8-A)
- RN2 pad 2: Net-(D8-Pad2) -> Net-(D1-A)
- RN2 pad 3: Net-(D7-Pad2) -> Net-(D2-A)
- RN2 pad 4: Net-(D6-Pad2) -> Net-(D3-A)
- RN2 pad 5: Net-(D5-Pad2) -> Net-(D4-A)
- RN2 pad 6: Net-(D4-Pad2) -> Net-(D5-A)
- RN2 pad 7: Net-(D3-Pad2) -> Net-(D6-A)
- RN2 pad 8: Net-(D2-Pad2) -> Net-(D7-A)
- RN2 pad 9: Net-(D1-Pad2) -> Net-(D8-A)
- U1 pad 11: Net-(D1-Pad2) -> Net-(D8-A)
- U1 pad 12: Net-(D2-Pad2) -> Net-(D7-A)
- U1 pad 13: Net-(D3-Pad2) -> Net-(D6-A)
- U1 pad 15: Net-(D4-Pad2) -> Net-(D5-A)
- U1 pad 16: Net-(D5-Pad2) -> Net-(D4-A)
- U1 pad 17: Net-(D6-Pad2) -> Net-(D3-A)
- U1 pad 18: Net-(D7-Pad2) -> Net-(D2-A)
- U1 pad 19: Net-(D8-Pad2) -> Net-(D1-A)
- U1 pad 20: GND -> A15
- U2 pad 10: Net-(U2-Pad10) -> unconnected-(U2-Pad10)
- U2 pad 11: Net-(R1-Pad1) -> GND
- U2 pad 12: Net-(R1-Pad1) -> GND
- U2 pad 13: Net-(U2-Pad13) -> unconnected-(U2-Pad13)
- U2 pad 8: Net-(R1-Pad1) -> GND
- U2 pad 9: Net-(R1-Pad1) -> GND
- U3 pad 2: Net-(D1-Pad2) -> Net-(D8-A)
- U3 pad 3: Net-(D2-Pad2) -> Net-(D7-A)
- U3 pad 4: Net-(D3-Pad2) -> Net-(D6-A)
- U3 pad 5: Net-(D4-Pad2) -> Net-(D5-A)
- U3 pad 6: Net-(D5-Pad2) -> Net-(D4-A)
- U3 pad 7: Net-(D6-Pad2) -> Net-(D3-A)
- U3 pad 8: Net-(D7-Pad2) -> Net-(D2-A)
- U3 pad 9: Net-(D8-Pad2) -> Net-(D1-A)
- U4 pad 10: Net-(R1-Pad1) -> A15
- U4 pad 11: Net-(U4-Pad11) -> unconnected-(U4-Pad11)
- U4 pad 12: Net-(R1-Pad1) -> GND
- U4 pad 13: Net-(R1-Pad1) -> GND
- U4 pad 4: Net-(R1-Pad1) -> GND
- U4 pad 5: Net-(R1-Pad1) -> GND
- U4 pad 6: Net-(U4-Pad6) -> unconnected-(U4-Pad6)
- U4 pad 8: Net-(U4-Pad8) -> ~{CART_CS}
- U4 pad 9: Net-(R1-Pad1) -> A15
Routing:
- net ~{CART_CS}: track 0.00 -> 178.8 mm, vias 0 -> 1
- net Net-(D4-A): track 0.00 -> 154.1 mm, vias 0 -> 1
- net Net-(D8-A): track 0.00 -> 115.7 mm, vias 0 -> 1
- net Net-(D7-A): track 0.00 -> 105.6 mm, vias 0 -> 1
- net A6: track 54.9 -> 156.4 mm, vias 0 -> 1
- net Net-(D6-A): track 0.00 -> 100.5 mm, vias 0 -> 1
- net Net-(D5-A): track 0.00 -> 94.0 mm
- net Net-(D3-A): track 0.00 -> 89.0 mm, vias 0 -> 4
- net Net-(D2-A): track 0.00 -> 81.2 mm, vias 0 -> 2
- net A15: track 53.8 -> 134.4 mm
- net A8: track 55.9 -> 134.3 mm
- net Net-(D3-Pad2): track 77.3 -> 0.00 mm, vias 2 -> 0
- net Net-(R1-Pad1): track 77.0 -> 0.00 mm
- net Net-(D1-Pad2): track 73.2 -> 0.00 mm
- net Net-(D2-Pad2): track 72.2 -> 0.00 mm, vias 1 -> 0
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Other:
- net class Default removed
- board text added: "Cartridge"
