File: Control Module/Control Module.kicad_pcb (KiCad board)
At the start: 2 copper layers, 99.6 x 99.6 mm, 73 parts, among them J1 USB_C_PowerOnly_6P, J2 Conn_01x22, J3 Conn_01x22, SW1 SW_Push, U1 74HC161, U11 74HC08, U12 74HC08, U13 74HC08, U2 74HC173, U3 74HC173, U4 28C256, U5 28C256, U6 74HC08, U7 74HC04, U8 74HC173, U9 74LS02

Commit message: Make Control Module 4 layers, and add 2 GND pins per side
Parts:
- J2, J3: value Conn_01x22 -> Conn_01x24; footprint Connector_PinSocket_2.54mm:PinSocket_1x22_P2.54mm_Horizontal -> Connector_PinSocket_2.54mm:PinSocket_1x24_P2.54mm_Horizontal
- moved J3 2.54 mm to (104.9, 41.7)
- moved J2 2.54 mm to (46.5, 119.9)
- moved C8 1.02 mm to (111.3, 123.8)
- moved U7 0.25 mm to (108.5, 42.2)
Connections:
- J2 pad 10: BOTTOM_SIG_OUT_2 -> BOTTOM_SIG_OUT_1
- J2 pad 11: CW12 -> BOTTOM_SIG_OUT_2
- J2 pad 12: CW13 -> CW12
- J2 pad 13: CW14 -> CW13
- J2 pad 14: CW15 -> CW14
- J2 pad 15: BUS0 -> CW15
- J2 pad 16: BUS1 -> BUS0
- J2 pad 17: BUS2 -> BUS1
- J2 pad 18: BUS3 -> BUS2
- J2 pad 19: BUS4 -> BUS3
- J2 pad 2: VCC -> GND
- J2 pad 20: BUS5 -> BUS4
- J2 pad 21: BUS6 -> BUS5
- J2 pad 22: BUS7 -> BUS6
- J2 pad 3: RESET -> VCC
- J2 pad 4: CLOCK -> RESET
- J2 pad 5: BOTTOM_SIG_IN_0 -> CLOCK
- J2 pad 6: BOTTOM_SIG_IN_1 -> BOTTOM_SIG_IN_0
- J2 pad 7: BOTTOM_SIG_IN_2 -> BOTTOM_SIG_IN_1
- J2 pad 8: BOTTOM_SIG_OUT_0 -> BOTTOM_SIG_IN_2
- J2 pad 9: BOTTOM_SIG_OUT_1 -> BOTTOM_SIG_OUT_0
- J3 pad 1: BUS7 -> GND
- J3 pad 10: CW10 -> CW11
- J3 pad 11: CW9 -> CW10
- J3 pad 12: CW8 -> CW9
- J3 pad 13: TOP_SIG_OUT_2 -> CW8
- J3 pad 14: TOP_SIG_OUT_1 -> TOP_SIG_OUT_2
- J3 pad 15: TOP_SIG_OUT_0 -> TOP_SIG_OUT_1
- J3 pad 16: TOP_SIG_IN_2 -> TOP_SIG_OUT_0
- J3 pad 17: TOP_SIG_IN_1 -> TOP_SIG_IN_2
- J3 pad 18: TOP_SIG_IN_0 -> TOP_SIG_IN_1
- J3 pad 19: CLOCK -> TOP_SIG_IN_0
- J3 pad 2: BUS6 -> BUS7
- J3 pad 20: RESET -> CLOCK
- J3 pad 21: VCC -> RESET
- J3 pad 22: GND -> VCC
- J3 pad 3: BUS5 -> BUS6
- J3 pad 4: BUS4 -> BUS5
- J3 pad 5: BUS3 -> BUS4
- J3 pad 6: BUS2 -> BUS3
- J3 pad 7: BUS1 -> BUS2
- J3 pad 8: BUS0 -> BUS1
- J3 pad 9: CW11 -> BUS0
Routing:
- net GND: track 527.4 -> 514.5 mm
- net BOTTOM_SIG_IN_0: track 165.9 -> 157.6 mm, vias 7 -> 5
- net VCC: track 446.6 -> 444.6 mm
- net TOP_SIG_IN_1: track 43.2 -> 44.4 mm
- net CLOCK: track 216.9 -> 217.9 mm
- net CW11: track 167.0 -> 166.0 mm
- net ~{CLOCK}: track 211.7 -> 212.3 mm
- added copper zone on In1.Cu, net GND
- added copper zone on In2.Cu, net GND
Other:
- copper layers 2 -> 4
- board text added: "Spork-8 Control board r3.1"
- board text removed: "Spork-8 Control board r3"
