File: Control Module/Control Module.kicad_sch (KiCad schematic)
At the start: 64 parts, among them J1 USB_C_PowerOnly_6P, SW1 SW_Push, U1 74HC161, U2 74HC173, U3 74HC173, U4 28C256, U5 28C256, U6 74HC08, U7 74HC04, U8 74HC173

Commit message: Make Control Module 4 layers, and add 2 GND pins per side
Parts:
- J1: LCSC (none) -> C2988369
